File: Rev-1/hardware/RO-Trng.kicad_sch (KiCad schematic)
At the start: 45 parts, among them J1 RFShield_OnePiece, J2 USB_C_Receptacle_USB2.0_14P, J3 TC2050, U1 74LVC04, U2 74LVC04, U3 74LVC04, U4 74HC174, U5 STM32F070F6Px, U6 AP2112K-3.3

Commit message: PCB update
Parts:
- added C17, C18: 12pF, Capacitor_SMD:C_0402_1005Metric, symbol Device:C_Small
- added R14: 10k, Resistor_SMD:R_0805_2012Metric, symbol Device:R_Small
- added SW1: SW_Push, Button_Switch_SMD:SW_Push_1P1T_XKB_TS-1187A, symbol Switch:SW_Push
- added Y1: 12Mhz, Crystal:Crystal_SMD_3225-4Pin_3.2x2.5mm, symbol Device:Crystal_Small
Connections:
- net GND: now also C17.1, C18.1, R14.1; no longer U5.1 (BOOT0)
- net VCC: now also SW1.2
- net OSC_IN: now reaches U5.2 (PF0)
- net OSC_IN: now also C17.2, Y1.2
- net OSC_OUT: now reaches U5.3 (PF1)
- net OSC_OUT: now also C18.2, Y1.1
- new net BOOT: R14.2, SW1.1, U5.1 (BOOT0)
Other:
- moved on the sheet: D1, R12

Commit message: update capacitors from 12 to 18pF
Parts:
- C17, C18: value 12pF -> 18pF
Changed lines of the file:
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@@
 			)
 		)
-		(property "Value" "12pF"
+		(property "Value" "18pF"
 			(at 185.4263 67.31 90)
 			(effects
@@
 			)
 		)
-		(property "Value" "12pF"
+		(property "Value" "18pF"
 			(at 185.4263 77.47 90)
 			(effects
