File: Rev-1/hardware/RO-Trng.kicad_pcb (KiCad board)
At the start: 2 copper layers, 41.6 x 48.7 mm, 45 parts, among them J1 RFShield_OnePiece, J2 USB_C_Receptacle_USB2.0_14P, J3 TC2050, U1 74LVC04, U2 74LVC04, U3 74LVC04, U4 74HC174, U5 STM32F070F6Px, U6 AP2112K-3.3

Commit message: PCB update
Parts:
- added C17: 12pF, Capacitor_SMD:C_0402_1005Metric, F.Cu at (127.0, 86.7)
- added C18: 12pF, Capacitor_SMD:C_0402_1005Metric, F.Cu at (127.0, 88.7)
- added R14: 10k, Resistor_SMD:R_0805_2012Metric, F.Cu at (128.6, 82.8)
- added SW1: SW_Push, Button_Switch_SMD:SW_Push_1P1T_XKB_TS-1187A, F.Cu at (123.2, 93.6)
- added Y1: 12Mhz, Crystal:Crystal_SMD_3225-4Pin_3.2x2.5mm, F.Cu at (124.5, 87.7)
- moved C11 20.9 mm to (144.6, 79.9)
- moved R1 20.9 mm to (144.6, 81.7)
- moved C13 15.2 mm to (107.8, 86.3), turned to 90 degrees
- moved R12 14.6 mm to (110.0, 82.4)
- moved D1 14.6 mm to (110.6, 81.0)
- moved R4 13.8 mm to (109.4, 87.0), turned to 90 degrees
- moved FB1 5.74 mm to (128.2, 95.0), turned to 90 degrees
Connections:
- U5 pad 1: GND -> /BOOT
- U5 pad 2: unconnected-(U5-PF0-Pad2) -> /OSC_IN
- U5 pad 3: unconnected-(U5-PF1-Pad3) -> /OSC_OUT
Routing:
- net /BOOT: track 0.00 -> 22.3 mm
- net GND: track 40.6 -> 55.0 mm, vias 107 -> 119
- net VCC: track 80.8 -> 94.1 mm
- net /NRST: track 27.0 -> 32.2 mm
- net /OSC_IN: track 0.00 -> 4.39 mm
- net /OSC_OUT: track 0.00 -> 4.29 mm
- net Net-(U5-VDDA): track 3.65 -> 6.73 mm
- net /D+: track 24.7 -> 27.5 mm
Other:
- board text removed: "PWR"

Commit message: Rev 2 of hardware
Parts:
- C17, C18: value 12pF -> 18pF
Changed lines of the file:
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@@
 			)
 		)
+		(property ki_fp_filters "C_*")
+		(sheetname "/")
+		(sheetfile "RO-Trng.kicad_sch")
 		(attr smd)
 		(fp_line
@@
 			)
 			(layer "F.SilkS")
-			(net 112)
 		)
 		(fp_line
@@
 			)
 			(layer "F.SilkS")
-			(net 112)
 		)
 		(fp_poly
@@
 			(fill no)
 			(layer "F.CrtYd")
-			(net 112)
 		)
 		(fp_poly
@@
 			(fill no)
 			(layer "F.Fab")
-			(net 112)
 		)
 		(fp_text user "${REFERENCE}"
@@
 			(at 0 -1.43 90)
 			(layer "F.SilkS")
+			(hide yes)
 			(effects
 				(font
@@
 			)
 		)
-		(property "Value" "12pF"
+		(property "Value" "18pF"
 			(at 0 1.16 90)
 			(layer "F.Fab")
@@
 			)
 		)
+		(property ki_fp_filters "R_*")
+		(sheetname "/")
+		(sheetfile "RO-Trng.kicad_sch")
 		(attr smd)
 		(fp_line
@@
 			)
 		)
+		(property ki_fp_filters "LED* LED_SMD:* LED_THT:*")
+		(sheetname "/")
+		(sheetfile "RO-Trng.kicad_sch")
 		(attr smd)
 		(fp_line
@@
 			)
 		)
+		(property ki_fp_filters "R_*")
+		(sheetname "/")
+		(sheetfile "RO-Trng.kicad_sch")
 		(attr smd)
 		(fp_line
@@
 			)
 			(layer "F.SilkS")
-			(net 112)
 		)
 		(fp_line
@@
 			)
 			(layer "F.SilkS")
-			(net 112)
 		)
 		(fp_poly
@@
 			(fill no)
 			(layer "F.CrtYd")
-			(net 112)
 		)
 		(fp_poly
@@
 			(fill no)
 			(layer "F.Fab")
-			(net 112)
 		)
 		(fp_text user "${REFERENCE}"
@@
 			)
 		)
-		(property "Value" "12pF"
+		(property "Value" "18pF"
 			(at 0 1.16 90)
 			(layer "F.Fab")
@@
 			)
 		)
-		(property "LCSC" "C1523"
+		(property "LCSC" "C1549"
 			(at 0 0 0)
 			(layer "F.SilkS")
